Commit message: add gazebo visualization

File: py2_amr/src/detection/models/AMR.xacro (robot description, xacro)
@@ -61,5 +61,5 @@
     <xacro:laser name="sensor_laser_back"/>
     <xacro:sensor_d435 name="camera" topics_ns="camera" parent="chassis" publish_pointcloud="true">
-        <origin xyz="0.51 0 -0.05" rpy="0 0 0" />
+        <origin xyz="0.51 0 0.155" rpy="0 0 0" />
     </xacro:sensor_d435>
     <!-- Joint -->

Commit message: final
detection - gazebo detection
show result -gui

File: py2_amr/src/detection/models/AMR.xacro (robot description, xacro)
@@ -61,5 +61,5 @@
     <xacro:laser name="sensor_laser_back"/>
     <xacro:sensor_d435 name="camera" topics_ns="camera" parent="chassis" publish_pointcloud="true">
-        <origin xyz="0.51 0 0.155" rpy="0 0 0" />
+        <origin xyz="0.51 0 0.155" rpy="0 -0.086 0" />
     </xacro:sensor_d435>
     <!-- Joint -->
